File: hardware/TCD1304/TCD1304.kicad_pcb (KiCad board)
At the start: 2 copper layers, 12 parts, among them J1 SUPPLY, J5 UART, J6 OUTPUT_STAGE, J7 JUMPER_ADC_BTJ, Q1 PNP

Commit message: pcb prototype
Parts:
- moved J1 2.00 mm to (208.5, 111.5)
Routing:
- net GND: track 171.5 -> 160.7 mm
- net +3.3V: track 125.0 -> 114.7 mm
Changed lines of the file:
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@@
 	(footprint "Connector_PinHeader_2.54mm:PinHeader_1x02_P2.54mm_Vertical"
 		(layer "F.Cu")
-		(at 206.5 111.5 180)
+		(at 208.5 111.5 180)
 		(descr "Through hole straight pin header, 1x02, 2.54mm pitch, single row")
 		(tags "Through hole pin header THT 1x02 2.54mm single row")
@@
 	)
 	(segment
-		(start 209 82.5)
-		(end 187.765 82.5)
-		(width 0.2)
-		(layer "F.Cu")
-		(net 1)
-	)
-	(segment
 		(start 170.3 115.58)
 		(end 172.84 115.58)
@@
 	)
 	(segment
-		(start 205 116.5)
-		(end 213.5 116.5)
+		(start 170 111.5)
+		(end 202.5 111.5)
 		(width 0.2)
 		(layer "F.Cu")
@@
 	)
 	(segment
-		(start 170 111.5)
-		(end 203.96 111.5)
-		(width 0.2)
-		(layer "F.Cu")
-		(net 1)
-	)
-	(segment
-		(start 203.96 111.5)
-		(end 206.5 108.96)
-		(width 0.2)
-		(layer "F.Cu")
-		(net 1)
-	)
-	(segment
-		(start 213.5 116.5)
-		(end 213.5 87)
+		(start 183.5 87.5)
+		(end 183.5 90)
+		(width 0.2)
+		(layer "F.Cu")
+		(net 1)
+	)
+	(segment
+		(start 204.5 85)
+		(end 208.5 89)
+		(width 0.2)
+		(layer "F.Cu")
+		(net 1)
+	)
+	(segment
+		(start 206 115)
+		(end 212.5 115)
+		(width 0.2)
+		(layer "F.Cu")
+		(net 1)
+	)
+	(segment
+		(start 184.5 85)
+		(end 204.5 85)
 		(width 0.2)
 		(layer "F.Cu")
@@
 	)
 	(segment
+		(start 208.5 89)
+		(end 208.5 108.96)
+		(width 0.2)
+		(layer "F.Cu")
+		(net 1)
+	)
+	(segment
+		(start 183.395 86.87)
+		(end 183.395 87.395)
+		(width 0.2)
+		(layer "F.Cu")
+		(net 1)
+	)
+	(segment
+		(start 212.5 115)
+		(end 212.5 110)
+		(width 0.2)
+		(layer "F.Cu")
+		(net 1)
+	)
+	(segment
 		(start 170 115.28)
 		(end 170.3 115.58)
@@
 	)
 	(segment
-		(start 213.5 87)
-		(end 209 82.5)
-		(width 0.2)
-		(layer "F.Cu")
-		(net 1)
-	)
-	(segment
-		(start 203.96 115.46)
-		(end 205 116.5)
-		(width 0.2)
-		(layer "F.Cu")
-		(net 1)
-	)
-	(segment
-		(start 203.96 111.5)
-		(end 203.96 115.46)
-		(width 0.2)
-		(layer "F.Cu")
-		(net 1)
-	)
-	(segment
-		(start 187.765 82.5)
-		(end 183.395 86.87)
-		(width 0.2)
-		(layer "F.Cu")
-		(net 1)
-	)
-	(segment
-		(start 208 110)
-		(end 206.5 111.5)
-		(width 0.2)
-		(layer "F.Cu")
-		(net 2)
-	)
-	(segment
-		(start 171.88 107)
-		(end 206.065 107)
-		(width 0.2)
-		(layer "F.Cu")
-		(net 2)
-	)
-	(segment
-		(start 206.065 107)
-		(end 208 107)
-		(width 0.2)
-		(layer "F.Cu")
-		(net 2)
-	)
-	(segment
-		(start 185.935 86.87)
-		(end 206.065 107)
+		(start 212.5 110)
+		(end 211.46 108.96)
+		(width 0.2)
+		(layer "F.Cu")
+		(net 1)
+	)
+	(segment
+		(start 183.395 86.105)
+		(end 184.5 85)
+		(width 0.2)
+		(layer "F.Cu")
+		(net 1)
+	)
+	(segment
+		(start 202.5 111.5)
+		(end 206 115)
+		(width 0.2)
+		(layer "F.Cu")
+		(net 1)
+	)
+	(segment
+		(start 183.395 87.395)
+		(end 183.5 87.5)
+		(width 0.2)
+		(layer "F.Cu")
+		(net 1)
+	)
+	(segment
+		(start 211.46 108.96)
+		(end 208.5 108.96)
+		(width 0.2)
+		(layer "F.Cu")
+		(net 1)
+	)
+	(segment
+		(start 183.395 86.87)
+		(end 183.395 86.105)
+		(width 0.2)
+		(layer "F.Cu")
+		(net 1)
+	)
+	(segment
+		(start 204 109)
+		(end 174 109)
 		(width 0.2)
 		(layer "F.Cu")
@@
 	)
 	(segment
+		(start 205.5 111.5)
+		(end 204 110)
+		(width 0.2)
+		(layer "F.Cu")
+		(net 2)
+	)
+	(segment
+		(start 208.5 111.5)
+		(end 205.5 111.5)
+		(width 0.2)
+		(layer "F.Cu")
+		(net 2)
+	)
+	(segment
 		(start 189.5 96)
 		(end 189.5 90.435)
@@
 	)
 	(segment
-		(start 208 107)
-		(end 208 110)
+		(start 204 110)
+		(end 204 109)
+		(width 0.2)
+		(layer "F.Cu")
+		(net 2)
+	)
+	(segment
+		(start 191 96)
+		(end 204 109)
 		(width 0.2)
 		(layer "F.Cu")
@@
 	)
 	(segment
+		(start 174 109)
+		(end 172 107)
+		(width 0.2)
+		(layer "F.Cu")
+		(net 2)
+	)
+	(segment
 		(start 157.92 129)
 		(end 157.92 136.42)
@@
 	)
 	(segment
+		(start 189.5 96)
+		(end 191 96)
+		(width 0.2)
+		(layer "F.Cu")
+		(net 2)
+	)
+	(segment
 		(start 194.825 143)
 		(end 202.695 135.13)
 		(width 0.2)
 		(layer "F.Cu")
+		(net 2)
+	)
+	(segment
+		(start 172 107)
+		(end 171.88 107)
+		(width 0.2)
+		(layer "F.Cu")
